File: hardware/V1.2/DIY_detector.kicad_pcb (KiCad board)
At the start: 2 copper layers, 75 x 26 mm, 35 parts, among them J1 Conn_01x02_Female, J2 Conn_01x02_Female, U1 TL072

Commit message: adding gerber files
Other:
- board text added: "α"
- board text added: "β"
- board text added: "μ"
Changed lines of the file:
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@@
   (general
     (thickness 1)
-    (drawings 56)
+    (drawings 59)
     (tracks 119)
     (zones 0)
@@
     (pad_to_mask_clearance 0.2)
     (aux_axis_origin 0 0)
-    (grid_origin 165.44 109.96)
+    (grid_origin 137.5 112.5)
     (visible_elements FFFFFE7F)
     (pcbplotparams
@@
       (net 4 GND))
   )
+  (gr_text μ (at 144.3072 112.5762 20) (layer F.Cu)
+    (effects (font (size 2 2) (thickness 0.3)))
+  )
+  (gr_text β (at 147.025 113.1604 -30) (layer F.Cu)
+    (effects (font (size 2 2) (thickness 0.3)))
+  )
+  (gr_text α (at 145.501 110.722 10) (layer F.Cu)
+    (effects (font (size 2 2) (thickness 0.3)))
+  )
   (gr_text B (at 160 122.5) (layer B.SilkS)
     (effects (font (size 1.5 1.5) (thickness 0.3)) (justify mirror))
@@
     (connect_pads thru_hole_only (clearance 0.2))
     (min_thickness 0.4)
-    (fill yes (arc_segments 16) (thermal_gap 0.4) (thermal_bridge_width 0.6))
+    (fill yes (arc_segments 16) (thermal_gap 0.4) (thermal_bridge_width 0.6) (smoothing chamfer) (radius 1))
     (polygon
       (pts
