File: hardware/V1.2/DIY_detector.kicad_pcb (KiCad board)
At the start: 2 copper layers, 75 x 26 mm, 35 parts, among them J1 Conn_01x02_Female, J2 Conn_01x02_Female, U1 TL072

Commit message: BOM files in preparation for Kitspace release
Parts:
- D1, D2, D3: value not populated -> see comments
- U1: value TL072 -> TLE2072
Changed lines of the file:
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@@
       (effects (font (size 1 1) (thickness 0.15)) (justify mirror))
     )
-    (fp_text value TL072 (at 3.81 -9.95) (layer B.Fab)
+    (fp_text value TLE2072 (at 3.81 -9.95) (layer B.Fab)
       (effects (font (size 1 1) (thickness 0.15)) (justify mirror))
     )
@@
       (effects (font (size 1 1) (thickness 0.15)))
     )
-    (fp_text value "not populated" (at 2.54 3.17 270) (layer F.Fab)
+    (fp_text value "see comments" (at 2.54 3.17 270) (layer F.Fab)
       (effects (font (size 1 1) (thickness 0.15)))
     )
@@
       (effects (font (size 1 1) (thickness 0.15)))
     )
-    (fp_text value "not populated" (at 1.27 3.17 90) (layer F.Fab)
+    (fp_text value "see comments" (at 1.27 3.17 90) (layer F.Fab)
       (effects (font (size 1 1) (thickness 0.15)))
     )
@@
       (effects (font (size 1 1) (thickness 0.15)))
     )
-    (fp_text value "not populated" (at 2.54 3.17 90) (layer F.Fab)
-      (effects (font (size 1 1) (thickness 0.15)))
-    )
+    (fp_text value "see comments" (at 2.54 3.17 90) (layer F.Fab)
+      (effects (font (size 1 1) (thickness 0.15)))
+    )

Commit message: renderings and 3D part models for both variants
including generated 3D models for all THT resistors, opamp chip model
with label. also created more accurate BPX61 TO-39 model.
Schematic and exported .xml BOM file have two new columns which store
part values and 3D model locations of the electron detector assembly
variant (VALUE_B, 3D_B)
Parts:
- D1: value see comments -> BPX61
- D2, D3: value see comments -> DNP
- D4: value BPX61 -> DNP
